Commit message: Add simulated Hesai XT16 LiDAR to Go2 URDF initial

File: ros2_ws/src/go2_description/urdf/go2.urdf (robot description, URDF)
Before this commit: robot go2_description, 42 links, 41 joints
Links:
- added link hesai_xt16, mass 0.9; collision cylinder length=0.07 radius=0.05; visual cylinder length=0.07 radius=0.05
Joints:
- added joint hesai_xt16_joint: type fixed, parent base, child hesai_xt16, origin xyz=0.0 0.0 0.15 rpy=0 0 0
